Commit message: Se exportó a URDF con valores investigados.

File: brazo_robotico/robotAssem3.SLDASM/urdf/robotAssem3.SLDASM.urdf (robot description, URDF)
Before this commit: robot robotAssem3.SLDASM, 5 links, 4 joints
Links:
- link base_link: mass 20.083 -> 20.485
- link link_1: mass 14.515 -> 14.805
- link link_2: mass 14.649 -> 14.929
- link link_3: mass 12.052 -> 12.293
- link link_4: mass 2.2191 -> 2.2635
Joints:
- removed joint link_5
- added joint joint_4: type revolute, parent link_3, child link_4, origin xyz=0 0 1.16 rpy=0 0 0, axis 1 0 0, limit lower=-3.14 upper=3.14 effort=17.6 velocity=5
- joint joint_1: axis 0 -1 0 -> 0 0 1; limit lower=0 upper=3.142 effort=300 velocity=3 -> lower=-3.14 upper=3.14 effort=96.8 velocity=3; origin xyz=0 0 0.16 rpy=-1.5708 0 -1.5708 -> xyz=0 0 0.496 rpy=1.5708 0 -1.5708
- joint joint_2: axis 0 0 -1 -> 1 0 0; limit lower=-1.57 upper=1.57 effort=200 velocity=3 -> lower=-3.14 upper=3.14 effort=66.4 velocity=3.5; origin xyz=0 -0.336 0 rpy=0 0 0 -> xyz=0 0 0.796 rpy=0 0 0
- joint joint_3: axis 0 0 -1 -> 1 0 0; limit lower=0 upper=3.142 effort=200 velocity=3 -> lower=-3.14 upper=3.14 effort=44.8 velocity=4; origin xyz=0 -0.5 0 rpy=0 0 0 -> xyz=0 0 1.02 rpy=0 0 0
