Commit message: Se corrigió el archivo URDF

File: src/robotAssem3.SLDASM/urdf/robotAssem3.SLDASM.urdf (robot description, URDF)
Before this commit: robot robotAssem3.SLDASM, 5 links, 4 joints
Joints:
- joint joint_1: axis 0 0 1 -> 0 1 0; origin xyz=0 0 0.496 rpy=1.5708 0 -1.5708 -> xyz=0 0 0.496 rpy=1.5708 0 0
- joint joint_2: axis 1 0 0 -> 0 0 1; limit lower=-3.14 upper=3.14 effort=66.4 velocity=3.5 -> lower=-1.57 upper=1.57 effort=66.4 velocity=3.5; origin xyz=0 0 0.796 rpy=0 0 0 -> xyz=0 0 0 rpy=0 0 -1.5708
- joint joint_3: axis 1 0 0 -> 0 0 1; limit lower=-3.14 upper=3.14 effort=44.8 velocity=4 -> lower=-0.7854 upper=2.3562 effort=44.8 velocity=4; origin xyz=0 0 1.02 rpy=0 0 0 -> xyz=-0.5 0 0 rpy=0 0 3.1416
- joint joint_4: axis 1 0 0 -> 0 0 1; limit lower=-3.14 upper=3.14 effort=17.6 velocity=5 -> lower=-1.57 upper=1.57 effort=17.6 velocity=5; origin xyz=0 0 1.16 rpy=0 0 0 -> xyz=0.145 -0.42746 0.01 rpy=0 0 0
